Commit message: complete: pendulum description package and the pendulum control package

File: pendulum_robot_description/urdf/gazebo.xacro (robot description, xacro)
@@ -1,14 +1,38 @@
 <?xml version="1.0"?>
 <robot xmlns:xacro="http://www.ros.org/wiki/xacro">
-    <gazebo>
-        <!-- <plugin filename="gz-ros2-control-system" name="gz_ros2_control::GazeboSimROS2ControlPlugin">
-        </plugin> -->
-        <plugin filename="gz-sim-joint-state-publisher-system" name="gz::sim::systems::JointStatePublisher">
-            <topic>joint_states</topic>
-            <joint_name>shoulder_lift_joint</joint_name>
-        </plugin>
-        <plugin filename="gz-sim-sensors-system" name="gz::sim::systems::Sensors">
-            <render_engine>ogre2</render_engine>
-        </plugin>
-    </gazebo>
+    <xacro:macro name="define_gazebo_plugins" params="activate_control">
+        <xacro:if value="${activate_control}">
+            <!-- ROS 2 Control -->
+            <ros2_control name="control" type="system">
+                <hardware>
+                    <plugin>gz_ros2_control/GazeboSimSystem</plugin>
+                </hardware>
+                <joint name="shoulder_lift_joint">
+                    <command_interface name="position"/>
+                    <command_interface name="velocity"/>
+                    <state_interface name="position"/>
+                    <state_interface name="velocity"/>
+                    <state_interface name="effort"/>
+                </joint>
+            </ros2_control>
+            <gazebo>
+                <plugin filename="gz_ros2_control-system" name="gz_ros2_control::GazeboSimROS2ControlPlugin">
+                    <parameters>$(find pendulum_robot_control)/config/simple_pendulum_controller.yaml</parameters>
+                </plugin>
+            </gazebo>
+        </xacro:if>
+        <gazebo>
+            <!-- <plugin filename="libign_ros2_control-system.so" name="ign_ros2_control::IgnitionROS2ControlPlugin">
+                <topic>joint_states</topic>
+                <joint_name>shoulder_lift_joint</joint_name>
+            </plugin> -->
+            <plugin filename="gz-sim-joint-state-publisher-system" name="gz::sim::systems::JointStatePublisher">
+                <topic>joint_states</topic>
+                <joint_name>shoulder_lift_joint</joint_name>
+            </plugin>
+            <plugin filename="gz-sim-sensors-system" name="gz::sim::systems::Sensors">
+                <render_engine>ogre2</render_engine>
+            </plugin>
+        </gazebo>
+    </xacro:macro>
 </robot>

File: pendulum_robot_description/urdf/kinematic_chain.xacro (robot description, xacro)
@@ -61,5 +61,6 @@
             <axis xyz="0 1 0"/>
             <limit velocity="${max_angular_velocity}" effort="${max_effort}"/>
-            <origin xyz="0 ${width/2.0+ball_radius} ${base_height-axle_offset}" rpy="0 0 0"/>
+            <origin xyz="0 ${width/2.0+ball_radius} ${base_height-axle_offset}" rpy="0 0.01 0"/>
+            <dynamics damping="0.1" friction="0.1"/>
         </joint>
         <joint name="ball_joint" type="fixed">

File: pendulum_robot_description/urdf/pendulum_robot.urdf.xacro (robot description, xacro)
@@ -2,4 +2,5 @@
 <robot xmlns:xacro="http://www.ros.org/wiki/xacro" name="pendulum_robot">
     <xacro:arg name="robot_parameters_file" default="$(find pendulum_robot_description)/config/parameters.yaml"/>
+    <xacro:arg name="activate_control" default="false"/>
     <xacro:include filename="$(find pendulum_robot_description)/urdf/kinematic_chain.xacro"/>
     <xacro:include filename="$(find pendulum_robot_description)/urdf/gazebo.xacro"/>
@@ -9,3 +10,6 @@
         config_params_file="$(arg robot_parameters_file)"
     />
+    <xacro:define_gazebo_plugins
+        activate_control="$(arg activate_control)"
+    />
 </robot>
